File: DS1245Y_FRAM.kicad_pcb (KiCad board)
At the start: 2 copper layers, 18.8 x 41.7 mm, 39 parts, among them J1 Conn_01x16, J2 Conn_01x16, U1 AMS1117, U2 FM28V100

Commit message: rev. 1
Connections:
- R15 pad 2: Net-(R15-Pad2) -> Net-(U1-Pad1)
- R16 pad 1: Net-(R15-Pad2) -> Net-(U1-Pad1)
- U1 pad 1: unconnected-(U1-Pad1) -> Net-(U1-Pad1)
Routing:
- net Net-(U1-Pad1): track 0.00 -> 10.8 mm, vias 0 -> 2
- net A15: track 20.1 -> 23.1 mm
- net Net-(R15-Pad2): track 1.48 -> 0.00 mm
Other:
- board text added: "DS1245Y replacement rev. 1 12/22 @qw3rtzuiop"
- board text removed: "DS1245Y replacement rev. 0 12/22 @qw3rtzuiop"
Changed lines of the file:
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@@
   (net 46 "DQ1")
   (net 47 "DQ2")
-  (net 48 "Net-(R15-Pad2)")
+  (net 48 "Net-(U1-Pad1)")
   (net 49 "~CE")
   (net 50 "A15")
@@
   (net 61 "DQ4")
   (net 62 "DQ3")
-  (net 63 "unconnected-(U1-Pad1)")
-  (net 64 "unconnected-(U2-Pad9)")
+  (net 63 "unconnected-(U2-Pad9)")
   (footprint "Capacitor_SMD:C_0805_2012Metric" (layer "F.Cu")
     (at 54.102 51.308 -90)
@@
     (fp_line (start -1 0.625) (end -1 -0.625) (layer "F.Fab") (width 0.1))
     (pad "1" smd roundrect (at -0.9125 0) (size 1.025 1.4) (layers "F.Cu" "F.Paste" "F.Mask") (roundrect_rratio 0.243902439)
-      (net 48 "Net-(R15-Pad2)") (pintype "passive"))
+      (net 48 "Net-(U1-Pad1)") (pintype "passive"))
     (pad "2" smd roundrect (at 0.9125 0) (size 1.025 1.4) (layers "F.Cu" "F.Paste" "F.Mask") (roundrect_rratio 0.243902439)
       (net 2 "GND") (pintype "passive"))
@@
       (net 3 "VDD") (pinfunction "VDD") (pintype "input"))
     (pad "9" smd roundrect (at -6.425 0.25 270) (size 1.55 0.3) (layers "F.Cu" "F.Paste" "F.Mask") (roundrect_rratio 0.25)
-      (net 64 "unconnected-(U2-Pad9)") (pinfunction "NC") (pintype "no_connect"))
+      (net 63 "unconnected-(U2-Pad9)") (pinfunction "NC") (pintype "no_connect"))
     (pad "10" smd roundrect (at -6.425 0.75 270) (size 1.55 0.3) (layers "F.Cu" "F.Paste" "F.Mask") (roundrect_rratio 0.25)
       (net 34 "A16") (pinfunction "A16") (pintype "input"))
@@
     (fp_line (start 1.85 -3.35) (end 1.85 3.35) (layer "F.Fab") (width 0.1))
     (pad "1" smd rect (at -3.15 -2.3 180) (size 2 1.5) (layers "F.Cu" "F.Paste" "F.Mask")
-      (net 63 "unconnected-(U1-Pad1)") (pinfunction "ADJ") (pintype "input"))
+      (net 48 "Net-(U1-Pad1)") (pinfunction "ADJ") (pintype "input"))
     (pad "2" smd rect (at 3.15 0 180) (size 2 3.8) (layers "F.Cu" "F.Paste" "F.Mask")
       (net 3 "VDD") (pinfunction "VO") (pintype "power_out"))
@@
       (net 3 "VDD") (pintype "passive"))
     (pad "2" smd roundrect (at 0.9125 0) (size 1.025 1.4) (layers "F.Cu" "F.Paste" "F.Mask") (roundrect_rratio 0.243902439)
-      (net 48 "Net-(R15-Pad2)") (pintype "passive"))
+      (net 48 "Net-(U1-Pad1)") (pintype "passive"))
     (model "${KICAD6_3DMODEL_DIR}/Resistor_SMD.3dshapes/R_0805_2012Metric.wrl"
       (offset (xyz 0 0 0))
@@
   )
   (gr_rect (start 49.53 49.53) (end 68.326 91.186) (layer "Edge.Cuts") (width 0.2) (fill none))
-  (gr_text "DS1245Y\nreplacement\nrev. 0 12/22\n@qw3rtzuiop" (at 53.594 86.36) (layer "F.SilkS")
+  (gr_text "DS1245Y\nreplacement\nrev. 1 12/22\n@qw3rtzuiop" (at 53.594 86.36) (layer "F.SilkS")
     (effects (font (size 1 1) (thickness 0.15)) (justify left))
   )
@@
   (segment (start 57.15 86.614) (end 56.0305 86.614) (width 0.25) (layer "B.Cu") (net 47))
   (segment (start 55.5225 60.706) (end 56.9995 60.706) (width 0.25) (layer "F.Cu") (net 48))
+  (segment (start 62.318 58.166) (end 62.332 58.18) (width 0.25) (layer "F.Cu") (net 48))
+  (segment (start 56.9995 60.706) (end 58.2035 59.502) (width 0.25) (layer "F.Cu") (net 48))
+  (segment (start 60.706 58.166) (end 62.318 58.166) (width 0.25) (layer "F.Cu") (net 48))
+  (segment (start 58.2035 59.502) (end 58.2035 56.642) (width 0.25) (layer "F.Cu") (net 48))
+  (via (at 58.2035 56.642) (size 0.8) (drill 0.4) (layers "F.Cu" "B.Cu") (net 48))
+  (via (at 60.706 58.166) (size 0.8) (drill 0.4) (layers "F.Cu" "B.Cu") (net 48))
+  (segment (start 59.182 56.642) (end 60.706 58.166) (width 0.25) (layer "B.Cu") (net 48))
+  (segment (start 58.2035 56.642) (end 59.182 56.642) (width 0.25) (layer "B.Cu") (net 48))
   (segment (start 61.468 80.01) (end 61.468 78.487006) (width 0.25) (layer "F.Cu") (net 49))
   (segment (start 61.17 81.355) (end 61.17 80.308) (width 0.25) (layer "F.Cu") (net 49))
@@
   (segment (start 59.182 70.612) (end 59.182 68.517) (width 0.25) (layer "F.Cu") (net 50))
   (via (at 59.182 70.612) (size 0.8) (drill 0.4) (layers "F.Cu" "B.Cu") (net 50))
-  (segment (start 62.0795 53.848) (end 59.182 56.7455) (width 0.25) (layer "B.Cu") (net 50))
-  (segment (start 59.182 56.7455) (end 59.182 70.612) (width 0.25) (layer "B.Cu") (net 50))
+  (segment (start 57.404 55.88) (end 57.912 55.372) (width 0.25) (layer "B.Cu") (net 50))
+  (segment (start 57.912 55.372) (end 60.5555 55.372) (width 0.25) (layer "B.Cu") (net 50))
+  (segment (start 57.404 57.15) (end 57.404 55.88) (width 0.25) (layer "B.Cu") (net 50))
+  (segment (start 59.182 58.928) (end 57.404 57.15) (width 0.25) (layer "B.Cu") (net 50))
+  (segment (start 59.182 70.612) (end 59.182 58.928) (width 0.25) (layer "B.Cu") (net 50))
+  (segment (start 60.5555 55.372) (end 62.0795 53.848) (width 0.25) (layer "B.Cu") (net 50))
   (segment (start 60.96 60.706) (end 60.039969 61.626031) (width 0.25) (layer "F.Cu") (net 51))
   (segment (start 60.17 67.536) (end 60.17 68.505) (width 0.25) (layer "F.Cu") (net 51))
