File: DS1245Y_FRAM.kicad_sch (KiCad schematic)
At the start: 39 parts, among them J1 Conn_01x16, J2 Conn_01x16, U1 AMS1117, U2 FM28V100

Commit message: rev. 1
Connections:
- net at R15.2, R16.1: now also U1.1 (ADJ)
Changed lines of the file:
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@@
   (junction (at 95.25 20.32) (diameter 0) (color 0 0 0 0)
   )
+  (junction (at 83.82 30.48) (diameter 0) (color 0 0 0 0)
+  )
   (junction (at 71.12 40.64) (diameter 0) (color 0 0 0 0)
   )
@@
     (stroke (width 0) (type default) (color 0 0 0 0))
   )
-  (wire (pts (xy 83.82 29.21) (xy 83.82 31.75))
+  (wire (pts (xy 83.82 29.21) (xy 83.82 30.48))
     (stroke (width 0) (type default) (color 0 0 0 0))
   )
@@
     (stroke (width 0) (type default) (color 0 0 0 0))
   )
+  (wire (pts (xy 83.82 30.48) (xy 83.82 31.75))
+    (stroke (width 0) (type default) (color 0 0 0 0))
+  )
   (wire (pts (xy 139.7 72.39) (xy 143.51 72.39))
     (stroke (width 0) (type default) (color 0 0 0 0))
@@
     (stroke (width 0) (type default) (color 0 0 0 0))
   )
+  (wire (pts (xy 72.39 27.94) (xy 72.39 30.48))
+    (stroke (width 0) (type default) (color 0 0 0 0))
+  )
   (wire (pts (xy 77.47 68.58) (xy 80.01 68.58))
     (stroke (width 0) (type default) (color 0 0 0 0))
@@
     (stroke (width 0) (type default) (color 0 0 0 0))
   )
+  (wire (pts (xy 72.39 30.48) (xy 83.82 30.48))
+    (stroke (width 0) (type default) (color 0 0 0 0))
+  )
